File: hardware/LSM303D.kicad_pcb (KiCad board)
At the start: 2 copper layers, 29 x 28.7 mm, 11 parts, among them U1 LSM303D

Commit message: fix footprint
Parts:
- LSM303D: renamed from U1; footprint Package_LGA:LGA-16_3x3mm_P0.5mm -> Package_LGA:LGA-16_3x3mm_P0.5mm_LayoutBorder3x5y
- moved R2 7.88 mm to (172.4, 109.2), turned to 90 degrees
- moved SDA 3.90 mm to (183.9, 110.2)
- moved SCL 3.80 mm to (184.0, 114.1)
- moved R1 3.38 mm to (167.3, 109.4)
- renumbered 3.3V to VCC
Connections:
- LSM303D pad 4: SDA -> SCL
- LSM303D pad 6: SCL -> SDA
- R1 pad 2: SDA -> SCL
- R2 pad 2: SCL -> SDA
Routing:
- net GND: track 88.2 -> 10.4 mm, vias 2 -> 6
- net 3.3V: track 75.8 -> 52.7 mm, vias 0 -> 2
- net SDA: track 25.7 -> 17.0 mm
- net SCL: track 17.0 -> 25.0 mm
- added copper zone on B.Cu, net GND
